File: schematic & PCB/droidbot_main_HW.brd (EAGLE design)
At the start: 100 x 80 mm, 5 parts

Commit message: minor changes
Parts:
- added PH1, PH2: A1060_34, photo-elements:T0-46-A10XX
- added R1, R2, R3, R4: (no value), eagle-ltspice:0204/7
- added R5: PC16D, piher:PC16D
Connections:
- new net N$15: R1.1, R2.2
- new net N$16: R1.2, R4.1
- new net N$17: PH1.2, R2.1
- new net N$18: PH1.1, R4.2
- net N$9: now also UC_LH_PORT.19
Changed lines of the file:
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@@
 <layer number="97" name="Info" color="7" fill="1" visible="no" active="no"/>
 <layer number="98" name="Guide" color="6" fill="1" visible="no" active="no"/>
+<layer number="99" name="SpiceOrder" color="5" fill="1" visible="no" active="no"/>
 <layer number="100" name="Wires" color="12" fill="1" visible="yes" active="yes"/>
 </layers>
@@
 <attribute name="OC_FARNELL" value="unknown" x="27.94" y="8.89" size="1.778" layer="27" rot="R180" display="off"/>
 </element>
+<element name="R1" library="eagle-ltspice" package="0204/7" value="" x="5.08" y="-3.81">
+<attribute name="SPICEMODEL" value="NONE" x="5.08" y="-3.81" size="1.778" layer="27" display="off"/>
+<attribute name="SPICEPREFIX" value="R" x="5.08" y="-3.81" size="1.778" layer="27" display="off"/>
+</element>
+<element name="R2" library="eagle-ltspice" package="0204/7" value="" x="5.08" y="-7.62">
+<attribute name="SPICEMODEL" value="NONE" x="5.08" y="-7.62" size="1.778" layer="27" display="off"/>
+<attribute name="SPICEPREFIX" value="R" x="5.08" y="-7.62" size="1.778" layer="27" display="off"/>
+</element>
+<element name="R3" library="eagle-ltspice" package="0204/7" value="" x="5.08" y="-11.43">
+<attribute name="SPICEMODEL" value="NONE" x="5.08" y="-11.43" size="1.778" layer="27" display="off"/>
+<attribute name="SPICEPREFIX" value="R" x="5.08" y="-11.43" size="1.778" layer="27" display="off"/>
+</element>
+<element name="R4" library="eagle-ltspice" package="0204/7" value="" x="5.08" y="-15.24">
+<attribute name="SPICEMODEL" value="NONE" x="5.08" y="-15.24" size="1.778" layer="27" display="off"/>
+<attribute name="SPICEPREFIX" value="R" x="5.08" y="-15.24" size="1.778" layer="27" display="off"/>
+</element>
+<element name="PH1" library="photo-elements" package="T0-46-A10XX" value="A1060_34" x="-6.35" y="-10.16"/>
+<element name="PH2" library="photo-elements" package="T0-46-A10XX" value="A1060_34" x="-15.24" y="-10.16"/>
+<element name="R5" library="piher" package="PC16D" value="PC16D" x="-29.21" y="29.21">
+<attribute name="MPN" value="" x="-29.21" y="29.21" size="1.778" layer="27" display="off"/>
+<attribute name="OC_NEWARK" value="unknown" x="-29.21" y="29.21" size="1.778" layer="27" display="off"/>
+<attribute name="MF" value="" x="-29.21" y="29.21" size="1.778" layer="27" display="off"/>
+<attribute name="OC_FARNELL" value="4453049" x="-29.21" y="29.21" size="1.778" layer="27" display="off"/>
+</element>
 </elements>
 <signals>
@@
 <wire x1="36.83" y1="8.89" x2="60.96" y2="33.02" width="0.4064" layer="16"/>
 <wire x1="60.96" y1="33.02" x2="60.96" y2="44.45" width="0.4064" layer="16"/>
+<contactref element="UC_LH_PORT" pad="19"/>
 <wire x1="60.96" y1="44.45" x2="43.18" y2="45.72" width="0" layer="19" extent="1-1"/>
+<wire x1="19.05" y1="45.72" x2="43.18" y2="45.72" width="0" layer="19" extent="1-1"/>
 </signal>
 <signal name="N$10">
@@
 <contactref element="MOTOR_DRIVER_RH_PORT" pad="1"/>
 </signal>
+<signal name="N$15">
+<contactref element="R2" pad="2"/>
+<contactref element="R1" pad="1"/>
+<wire x1="8.89" y1="-7.62" x2="1.27" y2="-3.81" width="0" layer="19" extent="1-1"/>
+</signal>
+<signal name="N$16">
+<contactref element="R1" pad="2"/>
+<contactref element="R4" pad="1"/>
+<wire x1="8.89" y1="-3.81" x2="1.27" y2="-15.24" width="0" layer="19" extent="1-1"/>
+</signal>
+<signal name="N$17">
+<contactref element="R2" pad="1"/>
+<contactref element="PH1" pad="2"/>
+<wire x1="1.27" y1="-7.62" x2="-4.65" y2="-10.16" width="0" layer="19" extent="1-1"/>
+</signal>
+<signal name="N$18">
+<contactref element="R4" pad="2"/>
+<contactref element="PH1" pad="1"/>
+<wire x1="8.89" y1="-15.24" x2="-8.05" y2="-10.16" width="0" layer="19" extent="1-1"/>
+</signal>
 </signals>
